Commit message: Updated inverseKinematics

File: urdf/thorvald_arm.urdf (robot description, URDF)
Before this commit: robot thorvald_arm, 5 links, 4 joints
Joints:
- joint joint1: origin xyz=0 0 0 rpy=1.5708 0 0.97926 -> xyz=0 0 0 rpy=1.5708 0 0
- joint joint2: origin xyz=0.32 0.12 0 rpy=0 0.534874357555222 3.14159265358979 -> xyz=0.32 0.12 0 rpy=0 0 3.14159265358979
- joint nozzle_joint: origin xyz=-0.32 -0.05 0 rpy=-1.5707963267949 0.857942850459156 3.14159265358979 -> xyz=-0.32 -0.05 0 rpy=-1.5707963267949 0 3.14159265358979

Commit message: commit

File: urdf/thorvald_arm.urdf (robot description, URDF)
Before this commit: robot thorvald_arm, 5 links, 4 joints
Joints:
- joint joint1: limit (none) -> effort=30 velocity=1.0
- joint joint2: limit (none) -> effort=30 velocity=1.0
- joint nozzle_joint: limit (none) -> effort=30 velocity=1.0
